Commit message: [MiniQuadrotor][simulation] Add rotor effort interfaces

File: robots/mini_quadrotor/urdf/robot.gazebo.xacro (robot description, xacro)
@@ -5,7 +5,21 @@
   <!-- robot urdf -->
   <xacro:include filename="$(find mini_quadrotor)/urdf/robot.urdf.xacro" />
+  <xacro:macro name="rotor_control_joint" params="id">
+    <joint name="rotor${id}">
+      <command_interface name="effort">
+        <param name="min">${min_force}</param>
+        <param name="max">${max_force}</param>
+      </command_interface>
+      <state_interface name="position">
+        <param name="initial_value">${0}</param>
+      </state_interface>
+      <state_interface name="velocity"/>
+      <state_interface name="effort"/>
+    </joint>
+  </xacro:macro>
   <ros2_control name="aerial_robot_sim_system" type="system">
     <hardware>
       <plugin>gz_ros2_control/AerialRobotHwSim</plugin>
+      <param name="m_f_rate">${m_f_rate}</param>
     </hardware>
     <joint name="dummy_joint">
@@ -20,4 +34,8 @@
       <state_interface name="effort"/>
     </joint>
+    <xacro:rotor_control_joint id="1"/>
+    <xacro:rotor_control_joint id="2"/>
+    <xacro:rotor_control_joint id="3"/>
+    <xacro:rotor_control_joint id="4"/>
     <sensor name="spinal_imu">
       <state_interface name="orientation.x"/>

File: robots/mini_quadrotor/urdf/robot.urdf.xacro (robot description, xacro)
@@ -10,5 +10,6 @@
   <xacro:property name="rotor_z" value="0.026" />
   <!-- dynamics -->
-  <m_f_rate value="-0.011" /> <!-- drag torque rate -->
+  <xacro:property name="m_f_rate" value="-0.011" /> <!-- drag torque rate -->
+  <m_f_rate value="${m_f_rate}" />
   <xacro:property name="max_force" value="8.0" /> <!-- [N] -->
   <xacro:property name="min_force" value="0.0" /> <!-- [N] -->

Commit message: [MiniQuadrotor][simulation] Restore rotor visual spin

File: robots/mini_quadrotor/urdf/robot.gazebo.xacro (robot description, xacro)
@@ -3,4 +3,5 @@
     xmlns:xacro="http://www.ros.org/wiki/xacro" name="mini_quadrotor" >
   <xacro:arg name="robot_name" default="mini_quadrotor" />
+  <xacro:arg name="rotor_visual_speed_rate" default="20.0" />
   <!-- robot urdf -->
   <xacro:include filename="$(find mini_quadrotor)/urdf/robot.urdf.xacro" />
@@ -22,4 +23,5 @@
       <plugin>gz_ros2_control/AerialRobotHwSim</plugin>
       <param name="m_f_rate">${m_f_rate}</param>
+      <param name="rotor_visual_speed_rate">$(arg rotor_visual_speed_rate)</param>
     </hardware>
     <joint name="dummy_joint">

File: robots/mini_quadrotor/urdf/robot.urdf.xacro (robot description, xacro)
@@ -5,4 +5,5 @@
   <baselink name="fc" />
   <thrust_link name="thrust" />
+  <xacro:arg name="rotor_joint_velocity_limit" default="10000.0" />
   <!-- kinematics [m] -->
   <xacro:property name="rotor_x" value="0.085" />
@@ -14,4 +15,5 @@
   <xacro:property name="max_force" value="8.0" /> <!-- [N] -->
   <xacro:property name="min_force" value="0.0" /> <!-- [N] -->
+  <xacro:property name="rotor_joint_velocity_limit" value="$(arg rotor_joint_velocity_limit)" />
   <!-- friction -->
   <xacro:macro name="damping_factor" params="link">
@@ -40,5 +42,5 @@
   <xacro:macro name="propeller_module" params="id x y z direction">
     <joint name="rotor${id}" type="continuous">
-      <limit effort="100.0" lower="${min_force}" upper="${max_force}" velocity="0.5"/>
+      <limit effort="100.0" lower="${min_force}" upper="${max_force}" velocity="${rotor_joint_velocity_limit}"/>
       <parent link="main_body"/>
       <child link="thrust${id}"/>
